Commit message: urdf model with Gps sensors integrated

File: src/rovers_descriptions/urdf/cyclairbot_frontsteer.xacro (robot description, xacro)
@@ -15,6 +15,4 @@
     <color rgba="0 1.0 1.0 1.0"/>
   </material>
-  <!-- Gazebo references-->
-  <xacro:include filename="$(find ackermann_vehicle_description)/urdf/cyclairbot/cyclairbot_gazebo.xacro"/>
   <!-- Main robot body-->
   <link name="base_footprint"/>

File: src/rovers_descriptions/urdf/cyclairbot_frontsteer_gazebo.xacro (robot description, xacro)
@@ -50,5 +50,5 @@
           <plugin name='imu_plugin' filename='libgazebo_ros_imu_sensor.so'>
               <topicName>imu_data</topicName>
-              <bodyName>imu_link</bodyName>
+              <bodyName>imu_lin</bodyName>
               <updateRateHZ>10.0</updateRateHZ>
               <gaussianNoise>0.0</gaussianNoise>
@@ -58,4 +58,34 @@
           <pose>0 0 0 0 0 0</pose>
       </sensor>
+    </gazebo>
+    <!-- Imu s -->
+    <gazebo reference="gps_left_baseplate">
+      <sensor name="gps_sensor1" type="gps">
+          <always_on>true</always_on>
+          <update_rate>10.0</update_rate>
+          <plugin name="left_gps_sim" filename="libgazebo_ros_gps_sensor.so">
+              <ros>
+                  <!-- <namespace>/br</namespace> -->
+                  <remapping>left_gps_sim/out:=gps_left</remapping>
+              </ros>
+              <frame_name>gps_left_baseplate</frame_name>
+          </plugin>
+      </sensor>
+    </gazebo>
+    <gazebo reference="gps_right_baseplate">
+        <sensor name="gps_sensor2" type="gps">
+            <always_on>true</always_on>
+            <update_rate>10.0</update_rate>
+            <plugin name="right_gps_sim" filename="libgazebo_ros_gps_sensor.so">
+                <ros>
+                    <!-- <namespace>/br</namespace> -->
+                    <remapping>right_gps_sim/out:=gps_right</remapping>
+                </ros>
+                <drift>5.0 5.0 5.0</drift>
+                <gaussian_noise>0.1 0.1 0.1</gaussian_noise>
+                <frame_name>gps_right_baseplate</frame_name>
+            </plugin>
+        </sensor>
+        <material>Gazebo/Grey</material>
     </gazebo>
     <!--

File: src/rovers_descriptions/urdf/cyclairbot_v2.xacro (robot description, xacro)
@@ -1,7 +1,7 @@
 <?xml version="1.0"?>
-<robot xmlns:xacro="http://ros.org/wiki/xacro" name="cyclairbot_urdf" >
+<robot xmlns:xacro="http://ros.org/wiki/xacro" name="cyclairbot_v2" >
   <!-- bring different parts of robots  -->
-  <xacro:include filename="$(find rovers_descriptions)/urdf/cyclairbot_gazebo.xacro"/>
-  <xacro:include filename="$(find rovers_descriptions)/urdf/cyclairbot_soft.urdf"/>
+  <xacro:include filename="$(find rovers_descriptions)/urdf/cyclairbot_frontsteer_gazebo.xacro"/>
+  <xacro:include filename="$(find rovers_descriptions)/urdf/cyclairbot_frontsteer.xacro"/>
   <!--Add Realsense D435i sensor -->
   <xacro:arg name="use_nominal_extrinsics" default="false" />
@@ -18,3 +18,12 @@
     <axis rpy="0 0 0" xyz="0 0 1"/>
   </joint>
+  <!--Add Gps sensor  -->
+  <xacro:arg name="gps_num" default="2" />
+  <xacro:include filename="$(find rovers_descriptions)/urdf/gpsbase.xacro"/>
+  <joint name="gps_bot" type="fixed">
+    <parent link="main_box"/>
+    <child link="linking_plate"/>
+    <origin xyz="-0.5 0 0.31" rpy="0 0 0"/>
+    <axis rpy="0 0 0" xyz="0 0 1"/>
+  </joint>
 </robot>
